File: kicad/controle_grel.kicad_sch (KiCad schematic)
At the start: 17 parts, among them J1 ESP01, J2 Barrel_Jack_Switch, Q1 BC337, U1 AMS1117-3.3

Commit message: pcb: corrigido lado do ams1117 (colocando no botton)
Other:
- company: (none) -> Tomaz
- title: (none) -> Controle GREL
Changed lines of the file:
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@@
 	(generator_version "9.0")
 	(paper "A4")
+	(title_block
+		(title "Controle GREL")
+		(date "2025-07-01")
+		(rev "v1")
+		(company "Tomaz")
+	)
 	(rectangle
 		(start 97.79 20.32)

Commit message: Consegui corroer a plaquinhaaaa
Parts:
- removed J2: Barrel_Jack_Switch, Connector_BarrelJack:BarrelJack_Horizontal, symbol Connector:Barrel_Jack_Switch
- J1: footprint Connector_PinSocket_2.54mm:PinSocket_2x04_P2.54mm_Vertical -> Connector_PinSocket_2.54mm:PinSocket_2x04_P2.54mm_Vertical_SMD
- Q1: footprint Package_TO_SOT_THT:TO-92_Inline -> Connector_PinHeader_2.54mm:PinHeader_1x03_P2.54mm_Horizontal
- R1, R2, R3, R4, R5, R6, R7, R8: footprint Resistor_THT:R_Axial_DIN0207_L6.3mm_D2.5mm_P7.62mm_Horizontal -> Resistor_SMD:R_1206_3216Metric
Connections:
- net +3V3: now also bDOWN1.1, bON-OFF1.1, bUP1.1; no longer R1.2, R3.2, R5.2
- net B_UP: now also J1.7 (Pin_7); no longer J1.2 (Pin_2)
- net GND: now also R1.2, R3.2, R5.2; no longer bDOWN1.1, bON-OFF1.1, bUP1.1
- net IR: now also J1.2 (Pin_2); no longer J1.7 (Pin_7)
- net at D1.2 (A), R4.2, R6.2: now also D2.2 (A), R7.2, R8.2
